Commit message: Corrected XML & URDF, updated interactive_ik and ik_generator

File: assets/panda_tray/panda_tray.urdf (robot description, URDF)
Before this commit: robot panda_tray, 10 links, 9 joints
Links:
- added link tray_frame, mass 0.001
Joints:
- added joint tray_frame_to_base: type fixed, parent tray_frame, child tray_base, origin xyz=0 0 0 rpy=0 0 0
- joint panda_tray_fixed: child tray_base -> tray_frame

Commit message: Update the env

File: assets/panda_tray/panda_tray.urdf (robot description, URDF)
Before this commit: robot panda_tray, 11 links, 10 joints
Links:
- link panda_link0: geometry collision mesh filename=assets/panda_tray/mesh/link0.obj; visual mesh filename=assets/panda_tray/mesh/link0.obj
- link panda_link1: geometry collision mesh filename=assets/panda_tray/mesh/link1.obj; visual mesh filename=assets/panda_tray/mesh/link1.obj
- link panda_link2: geometry collision mesh filename=assets/panda_tray/mesh/link2.obj; visual mesh filename=assets/panda_tray/mesh/link2.obj
- link panda_link3: geometry collision mesh filename=assets/panda_tray/mesh/link3.obj; visual mesh filename=assets/panda_tray/mesh/link3.obj
- link panda_link4: geometry collision mesh filename=assets/panda_tray/mesh/link4.obj; visual mesh filename=assets/panda_tray/mesh/link4.obj
- link panda_link5: geometry collision mesh filename=assets/panda_tray/mesh/link5.obj; visual mesh filename=assets/panda_tray/mesh/link5.obj
- link panda_link6: geometry collision mesh filename=assets/panda_tray/mesh/link6.obj; visual mesh filename=assets/panda_tray/mesh/link6.obj
- link panda_link7: geometry collision mesh filename=assets/panda_tray/mesh/link7.obj; visual mesh filename=assets/panda_tray/mesh/link7.obj
